Commit message: chore: update CMakeLists, urdf (Manual_fix, identified_joint), remove obsolete identified urdf

File: urdf/AR5-5_07R-W4C4A2_ Manual_fix.urdf (robot description, URDF)
Before this commit: robot AR5-5_07R-W4C4A2, 10 links, 9 joints
Links:
- link AR5-5_07R-W4C4A2_base: mass 0.001 -> None
- link world: mass 0.001 -> None

File: urdf/AR5-5_07R-W4C4A2_identified_joint.urdf (robot description, URDF)
Before this commit: robot AR5-5_07R-W4C4A2, 10 links, 9 joints
Joints:
- joint AR5-5_07R-W4C4A2_joint_2: origin xyz=0.0 0.0 0.1745 rpy=0 0 0 -> xyz=0.0 0.0 0.174522 rpy=0 0 0
- joint AR5-5_07R-W4C4A2_joint_3: origin xyz=0.0 0.0 0.314 rpy=0 0 0 -> xyz=0.0 0.0 0.314726 rpy=0 0 0
- joint AR5-5_07R-W4C4A2_joint_5: origin xyz=-0.01 0.0 0.272 rpy=0 0 0 -> xyz=-0.01 0.0 0.272656 rpy=0 0 0
- joint AR5-5_07R-W4C4A2_tcp_joint: origin xyz=0.0 0.0 0.097 rpy=0 0 0 -> xyz=0.0 0.0 0.0968883 rpy=0 0 0
