Commit message: docs: URDF与Pinocchio惯量绕质心约定 + step2写URDF用Inertia矩阵
- 新增 docs/06-URDF与Pinocchio惯量绕质心约定.tex
- C++/Python step2 写 URDF 时显式使用 Inertia 的 3x3 惯量矩阵（绕质心 I_C）
- 统一写入精度：.6f/.6e（C++ 6 位）
- 补充 docs 01-05、config、scripts 等

Made-with: Cursor

File: urdf/AR5-5_07R-W4C4A2_identified_joint.urdf (robot description, URDF)
Before this commit: robot AR5-5_07R-W4C4A2, 10 links, 9 joints
Links:
- link AR5-5_07R-W4C4A2_link1: mass 2.683 -> 2.683000
- link AR5-5_07R-W4C4A2_link2: mass 2.3 -> 2.300000
- link AR5-5_07R-W4C4A2_link3: mass 1.862 -> 1.853578
- link AR5-5_07R-W4C4A2_link4: mass 1.234 -> 1.226160
- link AR5-5_07R-W4C4A2_link5: mass 1.328 -> 1.314494
- link AR5-5_07R-W4C4A2_link6: mass 0.93 -> 0.916494
- link AR5-5_07R-W4C4A2_link7: mass 0.332 -> 0.318494
