Commit message: feat: MuJoCo XML 与动力学脚本更新
- AR5-5_07R-W4C4A2.xml: option/contact 全自碰撞排除, position 执行器 kp+timeconst+dampratio
- step1_mujoco: 默认使用改好 XML, 每 0.5s 打印各关节力矩
- step1_pinocchio/random_compare: 默认路径与接触诊断
- step2 辨识与 URDF 相关脚本与配置更新

Made-with: Cursor

File: scripts/AR5-5_07R-W4C4A2/AR5-5_07R-W4C4A2.urdf (robot description, URDF)
Before this commit: robot AR5-5_07R-W4C4A2, 10 links, 9 joints
Links:
- link AR5-5_07R-W4C4A2_base: geometry collision mesh filename=AR5-5_07R-W4C4A2_base.stl scale=0.001 0.001 0.001; visual mesh filename=AR5-5_07R-W4C4A2_base.stl scale=0.001 0.001 0.001
- link AR5-5_07R-W4C4A2_link1: geometry collision mesh filename=AR5-5_07R-W4C4A2_link1.stl scale=0.001 0.001 0.001; visual mesh filename=AR5-5_07R-W4C4A2_link1.stl scale=0.001 0.001 0.001
- link AR5-5_07R-W4C4A2_link2: geometry collision mesh filename=AR5-5_07R-W4C4A2_link2.stl scale=0.001 0.001 0.001; visual mesh filename=AR5-5_07R-W4C4A2_link2.stl scale=0.001 0.001 0.001
- link AR5-5_07R-W4C4A2_link3: geometry collision mesh filename=AR5-5_07R-W4C4A2_link3.stl scale=0.001 0.001 0.001; visual mesh filename=AR5-5_07R-W4C4A2_link3.stl scale=0.001 0.001 0.001
- link AR5-5_07R-W4C4A2_link4: geometry collision mesh filename=AR5-5_07R-W4C4A2_link4.stl scale=0.001 0.001 0.001; visual mesh filename=AR5-5_07R-W4C4A2_link4.stl scale=.001 0.001 0.001
- link AR5-5_07R-W4C4A2_link5: geometry collision mesh filename=AR5-5_07R-W4C4A2_link5.stl scale=0.001 0.001 0.001; visual mesh filename=AR5-5_07R-W4C4A2_link5.stl scale=0.001 0.001 0.001
- link AR5-5_07R-W4C4A2_link6: geometry collision mesh filename=AR5-5_07R-W4C4A2_link6.stl scale=0.001 0.001 0.001; visual mesh filename=AR5-5_07R-W4C4A2_link6.stl scale=0.001 0.001 0.001
- link AR5-5_07R-W4C4A2_link7: geometry collision mesh filename=AR5-5_07R-W4C4A2_link7.stl scale=0.001 0.001 0.001; visual mesh filename=AR5-5_07R-W4C4A2_link7.stl scale=0.001 0.001 0.001
